File: eagle/espthing.brd (EAGLE design)
At the start: 35.6 x 54.6 mm, 15 parts, among them IC2 LM1117-3.3, U1 MAX3232

Commit message: added bom
Parts:
- C3, C4, C5, C6: value (none) -> 1uF
Changed lines of the file:
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@@
 <attribute name="VALUE" x="-6.35" y="18.923" size="1.778" layer="27" ratio="10" rot="R90"/>
 </element>
-<element name="C3" library="rcl" library_urn="urn:adsk.eagle:library:334" package="C1206" package3d_urn="urn:adsk.eagle:package:23618/2" value="" x="12.7" y="38.1" smashed="yes" rot="R270">
+<element name="C3" library="rcl" library_urn="urn:adsk.eagle:library:334" package="C1206" package3d_urn="urn:adsk.eagle:package:23618/2" value="1uF" x="12.7" y="38.1" smashed="yes" rot="R270">
 <attribute name="NAME" x="13.97" y="39.37" size="1.27" layer="25" rot="R270"/>
 <attribute name="POPULARITY" value="54" x="12.7" y="38.1" size="1.778" layer="27" rot="R270" display="off"/>
@@
 <attribute name="VALUE" x="10.16" y="39.37" size="1.27" layer="27" rot="R270"/>
 </element>
-<element name="C4" library="rcl" library_urn="urn:adsk.eagle:library:334" package="C1206" package3d_urn="urn:adsk.eagle:package:23618/2" value="" x="12.7" y="32.385" smashed="yes" rot="R270">
+<element name="C4" library="rcl" library_urn="urn:adsk.eagle:library:334" package="C1206" package3d_urn="urn:adsk.eagle:package:23618/2" value="1uF" x="12.7" y="32.385" smashed="yes" rot="R270">
 <attribute name="NAME" x="13.97" y="33.655" size="1.27" layer="25" rot="R270"/>
 <attribute name="POPULARITY" value="54" x="12.7" y="32.385" size="1.778" layer="27" rot="R270" display="off"/>
@@
 <attribute name="VALUE" x="10.16" y="33.655" size="1.27" layer="27" rot="R270"/>
 </element>
-<element name="C5" library="rcl" library_urn="urn:adsk.eagle:library:334" package="C1206" package3d_urn="urn:adsk.eagle:package:23618/2" value="" x="19.685" y="44.45" smashed="yes" rot="R180">
+<element name="C5" library="rcl" library_urn="urn:adsk.eagle:library:334" package="C1206" package3d_urn="urn:adsk.eagle:package:23618/2" value="1uF" x="19.685" y="44.45" smashed="yes" rot="R180">
 <attribute name="NAME" x="20.955" y="43.18" size="1.27" layer="25" rot="R180"/>
 <attribute name="POPULARITY" value="54" x="19.685" y="44.45" size="1.778" layer="27" rot="R180" display="off"/>
@@
 <attribute name="VALUE" x="20.955" y="46.99" size="1.27" layer="27" rot="R180"/>
 </element>
-<element name="C6" library="rcl" library_urn="urn:adsk.eagle:library:334" package="C1206" package3d_urn="urn:adsk.eagle:package:23618/2" value="" x="12.6749625" y="26.58040625" smashed="yes" rot="R90">
+<element name="C6" library="rcl" library_urn="urn:adsk.eagle:library:334" package="C1206" package3d_urn="urn:adsk.eagle:package:23618/2" value="1uF" x="12.6749625" y="26.58040625" smashed="yes" rot="R90">
 <attribute name="NAME" x="11.4049625" y="25.31040625" size="1.27" layer="25" rot="R90"/>
 <attribute name="POPULARITY" value="54" x="12.6749625" y="26.58040625" size="1.778" layer="27" rot="R90" display="off"/>
